File: ESPHome/PCB/BlockDetection/CurrentLoop/currentLoop/currentLoop.kicad_sch (KiCad schematic)
At the start: 11 parts, among them J1 Conn_01x03_Pin, J2 Conn_01x02_Pin, J3 Conn_01x02_Pin, Q1 BC856, Q2 BC557, U1 PC817

Commit message: current loop
Parts:
- added C2: 100nF, symbol Device:C
- added R2: 10R, symbol Device:R
Connections:
- net at C1.1, D1.2 (A), D2.1 (K)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: now also C2.1
- net at D1.1 (K), D2.2 (A), J1.2 (Pin_2): now also R2.2; no longer Q1.1 (B)
- new net: C2.2, Q1.1 (B), R2.1
Other:
- moved on the sheet: C1, D3, J2, J3, Q1, Q2, R1, U1

Commit message: current
Parts:
- R1: value R -> 1K8
Other:
- moved on the sheet: J2, J3, U1
Changed lines of the file:
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@@
 	)
 	(junction
-		(at 120.65 102.87)
-		(diameter 0)
-		(color 0 0 0 0)
-	)
-	(junction
-		(at 146.05 102.87)
-		(diameter 0)
-		(color 0 0 0 0)
-	)
-	(junction
-		(at 120.65 100.33)
+		(at 135.89 101.6)
 		(diameter 0)
 		(color 0 0 0 0)
@@
 	)
 	(junction
+		(at 157.48 101.6)
+		(diameter 0)
+		(color 0 0 0 0)
+	)
+	(junction
 		(at 106.68 59.69)
 		(diameter 0)
@@
 	)
 	(junction
-		(at 91.44 59.69)
+		(at 135.89 104.14)
 		(diameter 0)
 		(color 0 0 0 0)
 	)
 	(junction
-		(at 146.05 100.33)
+		(at 157.48 104.14)
+		(diameter 0)
+		(color 0 0 0 0)
+	)
+	(junction
+		(at 91.44 59.69)
 		(diameter 0)
 		(color 0 0 0 0)
@@
 	(wire
 		(pts
+			(xy 78.74 64.77) (xy 78.74 104.14)
+		)
+		(stroke
+			(width 0)
+			(type default)
+		)
+	)
+	(wire
+		(pts
 			(xy 116.84 78.74) (xy 124.46 78.74)
 		)
@@
 	(wire
 		(pts
-			(xy 120.65 100.33) (xy 146.05 100.33)
+			(xy 135.89 101.6) (xy 157.48 101.6)
 		)
 		(stroke
@@
 	(wire
 		(pts
-			(xy 116.84 100.33) (xy 120.65 100.33)
-		)
-		(stroke
-			(width 0)
-			(type default)
-		)
-	)
-	(wire
-		(pts
-			(xy 151.13 105.41) (xy 151.13 102.87)
+			(xy 162.56 106.68) (xy 162.56 104.14)
 		)
 		(stroke
@@
 	(wire
 		(pts
-			(xy 153.67 105.41) (xy 151.13 105.41)
+			(xy 165.1 106.68) (xy 162.56 106.68)
 		)
 		(stroke
@@
 	(wire
 		(pts
-			(xy 146.05 100.33) (xy 153.67 100.33)
+			(xy 78.74 104.14) (xy 135.89 104.14)
+		)
+		(stroke
+			(width 0)
+			(type default)
+		)
+	)
+	(wire
+		(pts
+			(xy 157.48 101.6) (xy 165.1 101.6)
 		)
 		(stroke
@@
 	(wire
 		(pts
-			(xy 74.93 102.87) (xy 120.65 102.87)
-		)
-		(stroke
-			(width 0)
-			(type default)
-		)
-	)
-	(wire
-		(pts
 			(xy 74.93 62.23) (xy 81.28 62.23)
 		)
@@
 	(wire
 		(pts
-			(xy 74.93 102.87) (xy 74.93 64.77)
+			(xy 116.84 101.6) (xy 135.89 101.6)
 		)
 		(stroke
@@
 	(wire
 		(pts
-			(xy 146.05 102.87) (xy 151.13 102.87)
+			(xy 157.48 104.14) (xy 162.56 104.14)
 		)
 		(stroke
@@
 	(wire
 		(pts
+			(xy 116.84 101.6) (xy 116.84 97.79)
+		)
+		(stroke
+			(width 0)
+			(type default)
+		)
+	)
+	(wire
+		(pts
 			(xy 91.44 59.69) (xy 106.68 59.69)
 		)
@@
 	(wire
 		(pts
-			(xy 120.65 102.87) (xy 146.05 102.87)
+			(xy 74.93 64.77) (xy 78.74 64.77)
+		)
+		(stroke
+			(width 0)
+			(type default)
+		)
+	)
+	(wire
+		(pts
+			(xy 135.89 104.14) (xy 157.48 104.14)
 		)
 		(stroke
@@
 		(pts
 			(xy 81.28 62.23) (xy 81.28 72.39)
-		)
-		(stroke
-			(width 0)
-			(type default)
-		)
-	)
-	(wire
-		(pts
-			(xy 116.84 100.33) (xy 116.84 97.79)
 		)
 		(stroke
@@
 			)
 		)
-		(property "Value" "R"
+		(property "Value" "1K8"
 			(at 119.38 86.3599 0)
 			(show_name no)
@@
 	(symbol
 		(lib_id "Isolator:PC817")
-		(at 161.29 102.87 0)
+		(at 172.72 104.14 0)
 		(unit 1)
 		(body_style 1)
@@
 		(fields_autoplaced yes)
 		(property "Reference" "U1"
-			(at 161.29 93.98 0)
+			(at 172.72 95.25 0)
 			(show_name no)
 			(do_not_autoplace no)
@@
 		)
 		(property "Value" "PC817"
-			(at 161.29 96.52 0)
+			(at 172.72 97.79 0)
 			(show_name no)
 			(do_not_autoplace no)
@@
 		)
 		(property "Footprint" "Package_DIP:DIP-4_W7.62mm"
-			(at 156.21 107.95 0)
+			(at 167.64 109.22 0)
 			(hide yes)
 			(show_name no)
@@
 		)
 		(property "Datasheet" "http://www.soselectronic.cz/a_info/resource/d/pc817.pdf"
-			(at 161.29 102.87 0)
+			(at 172.72 104.14 0)
 			(hide yes)
 			(show_name no)
@@
 		)
 		(property "Description" "DC Optocoupler, Vce 35V, CTR 50-300%, DIP-4"
-			(at 161.29 102.87 0)
+			(at 172.72 104.14 0)
 			(hide yes)
 			(show_name no)
@@
 	(symbol
 		(lib_id "Connector:Conn_01x02_Pin")
-		(at 125.73 100.33 0)
+		(at 140.97 101.6 0)
 		(mirror y)
 		(unit 1)
@@
 		(dnp no)
 		(property "Reference" "J3"
-			(at 125.476 105.41 0)
+			(at 140.716 106.68 0)
 			(show_name no)
 			(do_not_autoplace no)
@@
 		)
 		(property "Value" "Conn_01x02_Pin"
-			(at 125.095 97.79 0)
+			(at 140.335 99.06 0)
 			(hide yes)
 			(show_name no)
@@
 		)
 		(property "Footprint" ""
-			(at 125.73 100.33 0)
+			(at 140.97 101.6 0)
 			(hide yes)
 			(show_name no)
@@
 		)
 		(property "Datasheet" ""
-			(at 125.73 100.33 0)
+			(at 140.97 101.6 0)
 			(hide yes)
 			(show_name no)
@@
 		)
 		(property "Description" "Generic connector, single row, 01x02, script generated"
-			(at 125.73 100.33 0)
+			(at 140.97 101.6 0)
 			(hide yes)
 			(show_name no)
@@
 	(symbol
 		(lib_id "Connector:Conn_01x02_Pin")
-		(at 140.97 100.33 0)
+		(at 152.4 101.6 0)
 		(unit 1)
 		(body_style 1)
@@
 		(dnp no)
 		(property "Reference" "J2"
-			(at 141.224 105.156 0)
+			(at 152.654 106.426 0)
 			(show_name no)
 			(do_not_autoplace no)
@@
 		)
 		(property "Value" "Conn_01x02_Pin"
-			(at 141.605 97.79 0)
+			(at 153.035 99.06 0)
 			(hide yes)
 			(show_name no)
@@
 		)
 		(property "Footprint" ""
-			(at 140.97 100.33 0)
+			(at 152.4 101.6 0)
 			(hide yes)
 			(show_name no)
@@
 		)
 		(property "Datasheet" ""
-			(at 140.97 100.33 0)
+			(at 152.4 101.6 0)
 			(hide yes)
 			(show_name no)
@@
 		)
 		(property "Description" "Generic connector, single row, 01x02, script generated"
-			(at 140.97 100.33 0)
-			(hide yes)
-			(show_name no)
+			(at 152.4 101.6 0)
+			(hide yes)
+			(show_name no)

Commit message: current loop
Parts:
- removed Q2: BC557, Package_TO_SOT_THT:TO-92_Inline, symbol Transistor_BJT:BC557
- Q1: value BC856 -> BC856 or BC557
Changed lines of the file:
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@@
-	)
-	(symbol
-		(lib_id "Transistor_BJT:BC557")
-		(at 147.32 72.39 0)
-		(mirror x)
-		(unit 1)
-		(body_style 1)
-		(exclude_from_sim no)
-		(in_bom yes)
-		(on_board yes)
-		(in_pos_files yes)
-		(dnp no)
-		(property "Reference" "Q2"
-			(at 152.4 71.1199 0)
-			(show_name no)
-			(do_not_autoplace no)
-			(effects
-				(font
-					(size 1.27 1.27)
-				)
-				(justify left)
-			)
-		)
-		(property "Value" "BC557"
-			(at 152.4 73.6599 0)
-			(show_name no)
-			(do_not_autoplace no)
-			(effects
-				(font
-					(size 1.27 1.27)
-				)
-				(justify left)
-			)
-		)
-		(property "Footprint" "Package_TO_SOT_THT:TO-92_Inline"
-			(at 152.4 70.485 0)
-			(hide yes)
-			(show_name no)
-			(do_not_autoplace no)
-			(effects
-				(font
-					(size 1.27 1.27)
-					(italic yes)
-				)
-				(justify left)
-			)
-		)
-		(property "Datasheet" "https://www.onsemi.com/pub/Collateral/BC556BTA-D.pdf"
-			(at 147.32 72.39 0)
-			(hide yes)
-			(show_name no)
-			(do_not_autoplace no)
-			(effects
-				(font
-					(size 1.27 1.27)
-				)
-				(justify left)
-			)
-		)
-		(property "Description" "0.1A Ic, 45V Vce, PNP Small Signal Transistor, TO-92"
-			(at 147.32 72.39 0)
-			(hide yes)
-			(show_name no)
-			(do_not_autoplace no)
-			(effects
-				(font
-					(size 1.27 1.27)
-				)
-			)
-		)
-		(property "Sim.Device" "PNP"
-			(at 147.32 72.39 0)
-			(hide yes)
-			(show_name no)
-			(do_not_autoplace no)
-			(effects
-				(font
-					(size 1.27 1.27)
-				)
-			)
-		)
-		(property "Sim.Pins" "1=C 2=B 3=E"
-			(at 147.32 72.39 0)
-			(hide yes)
-			(show_name no)
-			(do_not_autoplace no)
-			(effects
-				(font
-					(size 1.27 1.27)
-				)
-			)
-		)
-		(pin "3"
-		)
-		(pin "1"
-		)
-		(pin "2"
-		)
-		(instances
-			(project "currentLoop"
-				(path "/df40a3ed-29e1-4fed-8bb8-557e0f8da153"
-					(reference "Q2")
-					(unit 1)
-				)
-			)
-		)
 	)
 	(symbol
@@
 			)
 		)
-		(property "Value" "BC856"
-			(at 117.856 66.548 0)
-			(show_name no)
-			(do_not_autoplace no)
+		(property "Value" "BC856 or BC557"
+			(at 109.474 56.896 0)
+			(show_name no)
+			(do_not_autoplace no)
